File: schematic/server/server.brd (EAGLE design)
At the start: 130 x 70 mm, 28 parts

Commit message: pinoutChange
Parts:
- moved DISPLAY 2.54 mm to (19.1, 61.0)
Connections:
- removed net N$20: ARDUINO-2.9, DISPLAY.3
- removed net N$21: ARDUINO-2.8, DISPLAY.4
- new net N$10: ARDUINO-2.9, DISPLAY.4
- new net N$8: ARDUINO-2.8, DISPLAY.3
- net GND: now also DISPLAY.1; no longer DISPLAY.2
- net N$18: now also DISPLAY.2; no longer DISPLAY.1
Routing:
- net GND: track 102.5 -> 340.4 mm
- net N$4: track 20.8 -> 140.0 mm
- net N$7: track 2.54 -> 84.0 mm, vias 0 -> 2
- net N$18: track 118.5 -> 189.8 mm
- net N$19: track 0.00 -> 71.0 mm
- net N$2: track 0.00 -> 61.6 mm
- net N$17: track 0.00 -> 52.2 mm
- net N$16: track 0.00 -> 42.7 mm
- net N$9: track 0.00 -> 33.3 mm
- net N$6: track 0.00 -> 23.9 mm
- net N$8: track 0.00 -> 13.8 mm
- net N$15: track 0.00 -> 9.72 mm
- net N$11: track 0.00 -> 6.35 mm
- net N$10: track 0.00 -> 5.08 mm
- net N$14: track 0.00 -> 3.81 mm
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